Commit message: feat: added more joints definitions

File: urdf/xarm.urdf (robot description, URDF)
Before this commit: robot xarm-lite-6, 8 links, 7 joints
Joints:
- joint base_link1_joint: limit lower=-3.14 upper=3.14 effort=0.0 velocity=0.0 -> (none); type revolute -> continuous
- joint gripper_link6_joint: axis (none) -> 0 0 1; type fixed -> continuous
- joint link1_link2_joint: axis (none) -> 0 0 1; limit (none) -> lower=-2.02 upper=2.02 effort=0.0 velocity=0.0; type fixed -> revolute
- joint link2_link3_joint: limit lower=0 upper=3.14 effort=0.0 velocity=0.0 -> lower=-0.06 upper=5.24 effort=0.0 velocity=0.0
- joint link3_link4_joint: axis (none) -> 0 0 1; origin xyz=0.1 -0.03 0.026 rpy=1.54 6.5 0.0 -> xyz=0.09 -0.03 0.008 rpy=1.5 6.4 0; type fixed -> continuous
- joint link4_link5_joint: axis (none) -> 0 0 1; limit (none) -> lower=-2.16 upper=2.16 effort=0.0 velocity=0.0; type fixed -> revolute
- joint link5_link6_joint: axis (none) -> 0 0 1
